File: pcb/pcb.kicad_pcb (KiCad board)
At the start: 2 copper layers, 350 x 170 mm, 0 parts

Commit message: Component placement
Parts:
- added D1: POWER, Sony_Hit_Bit:LED, F.Cu at (365.1, 104.0)
- added J1: Conn_01x24, Sony_Hit_Bit:Connector, F.Cu at (300.3, 61.5)
- added SW1: 0, Sony_Hit_Bit:Switch, F.Cu at (241.1, 124.4)
- added SW10: 9, Sony_Hit_Bit:Switch, F.Cu at (222.1, 124.4)
- added SW11: HYPHEN, Sony_Hit_Bit:Switch, F.Cu at (260.1, 124.4)
- added SW12: CARET, Sony_Hit_Bit:Switch, F.Cu at (279.2, 124.4)
- added SW13: YEN, Sony_Hit_Bit:Switch, F.Cu at (298.2, 124.4)
- added SW14: @, Sony_Hit_Bit:Switch, F.Cu at (270.3, 143.4)
- added SW15: [, Sony_Hit_Bit:Switch, F.Cu at (289.3, 143.4)
- added SW16: SEMICOLON, Sony_Hit_Bit:Switch, F.Cu at (255.9, 162.5)
- added SW17: COLON, Sony_Hit_Bit:Switch, F.Cu at (275.0, 162.5)
- added SW18: ], Sony_Hit_Bit:Switch, F.Cu at (294.0, 162.5)
- added SW19: COMMA, Sony_Hit_Bit:Switch, F.Cu at (227.4, 181.6)
- added SW2: 1, Sony_Hit_Bit:Switch, F.Cu at (69.7, 124.4)
- added SW20: FULLSTOP, Sony_Hit_Bit:Switch, F.Cu at (246.4, 181.6)
- added SW21: /, Sony_Hit_Bit:Switch, F.Cu at (265.5, 181.6)
- added SW22: UNDERSCORE, Sony_Hit_Bit:Switch, F.Cu at (284.5, 181.6)
- added SW23: A, Sony_Hit_Bit:Switch, F.Cu at (84.5, 162.5)
- added SW24: B, Sony_Hit_Bit:Switch, F.Cu at (170.2, 181.6)
- added SW25: C, Sony_Hit_Bit:Switch, F.Cu at (132.1, 181.6)
- added SW26: D, Sony_Hit_Bit:Switch, F.Cu at (122.6, 162.5)
- added SW27: E, Sony_Hit_Bit:Switch, F.Cu at (117.9, 143.4)
- added SW28: F, Sony_Hit_Bit:Switch, F.Cu at (141.6, 162.5)
- added SW29: G, Sony_Hit_Bit:Switch, F.Cu at (160.7, 162.5)
- added SW3: 2, Sony_Hit_Bit:Switch, F.Cu at (88.7, 124.4)
- added SW30: H, Sony_Hit_Bit:Switch, F.Cu at (179.7, 162.5)
- added SW31: I, Sony_Hit_Bit:Switch, F.Cu at (213.1, 143.4)
- added SW32: J, Sony_Hit_Bit:Switch, F.Cu at (198.8, 162.5)
- added SW33: K, Sony_Hit_Bit:Switch, F.Cu at (217.8, 162.5)
- added SW34: L, Sony_Hit_Bit:Switch, F.Cu at (236.9, 162.5)
- added SW35: M, Sony_Hit_Bit:Switch, F.Cu at (208.3, 181.6)
- added SW36: N, Sony_Hit_Bit:Switch, F.Cu at (189.3, 181.6)
- added SW37: O, Sony_Hit_Bit:Switch, F.Cu at (232.2, 143.4)
- added SW38: P, Sony_Hit_Bit:Switch, F.Cu at (251.2, 143.4)
- added SW39: Q, Sony_Hit_Bit:Switch, F.Cu at (79.8, 143.4)
- added SW4: 3, Sony_Hit_Bit:Switch, F.Cu at (107.8, 124.4)
- added SW40: R, Sony_Hit_Bit:Switch, F.Cu at (136.9, 143.4)
- added SW41: PAUSE, Sony_Hit_Bit:Switch, F.Cu at (306.0, 200.6)
- added SW42: S, Sony_Hit_Bit:Switch, F.Cu at (103.5, 162.5)
- added SW43: T, Sony_Hit_Bit:Switch, F.Cu at (156.0, 143.4)
- added SW44: U, Sony_Hit_Bit:Switch, F.Cu at (194.1, 143.4)
- added SW45: V, Sony_Hit_Bit:Switch, F.Cu at (151.2, 181.6)
- added SW46: W, Sony_Hit_Bit:Switch, F.Cu at (98.8, 143.4)
- added SW47: X, Sony_Hit_Bit:Switch, F.Cu at (113.1, 181.6)
- added SW48: Y, Sony_Hit_Bit:Switch, F.Cu at (175.0, 143.4)
- added SW49: Z, Sony_Hit_Bit:Switch, F.Cu at (94.0, 181.6)
- added SW5: 4, Sony_Hit_Bit:Switch, F.Cu at (126.8, 124.4)
- added SW50: LSHIFT, Sony_Hit_Bit:Switch, F.Cu at (63.0, 181.6)
- added SW51: CTRL, Sony_Hit_Bit:Switch, F.Cu at (58.3, 162.5)
- added SW52: GRAPH, Sony_Hit_Bit:Switch, F.Cu at (115.4, 200.6)
- added SW53: CAP, Sony_Hit_Bit:Switch, F.Cu at (89.2, 200.6)
- added SW54: KANA, Sony_Hit_Bit:Switch, F.Cu at (255.9, 200.6)
- added SW55: F1, Sony_Hit_Bit:Switch, F.Cu at (59.9, 104.0)
- added SW56: F2, Sony_Hit_Bit:Switch, F.Cu at (89.4, 104.0)
- added SW57: F3, Sony_Hit_Bit:Switch, F.Cu at (118.9, 104.0)
- added SW58: RSHIFT, Sony_Hit_Bit:Switch, F.Cu at (310.7, 181.6)
- added SW59: F4, Sony_Hit_Bit:Switch, F.Cu at (148.4, 104.0)
- added SW6: 5, Sony_Hit_Bit:Switch, F.Cu at (145.8, 124.4)
- added SW60: F5, Sony_Hit_Bit:Switch, F.Cu at (177.9, 104.0)
- added SW61: ESC, Sony_Hit_Bit:Switch, F.Cu at (51.1, 124.4)
- added SW62: TAB, Sony_Hit_Bit:Switch, F.Cu at (55.9, 143.4)
- added SW63: STOP, Sony_Hit_Bit:Switch, F.Cu at (313.1, 104.0)
- added SW64: BS, Sony_Hit_Bit:Switch, F.Cu at (317.3, 124.4)
- added SW65: SELECT, Sony_Hit_Bit:Switch, F.Cu at (280.4, 200.6)
- added SW66: RETURN, Sony_Hit_Bit:Switch, F.Cu at (315.5, 153.0)
- added SW67: SPACE, Sony_Hit_Bit:Switch, F.Cu at (189.3, 200.6)
- added SW68: HOME, Sony_Hit_Bit:Switch, F.Cu at (218.2, 104.0)
- added SW69: INS, Sony_Hit_Bit:Switch, F.Cu at (247.7, 104.0)
- added SW7: 6, Sony_Hit_Bit:Switch, F.Cu at (164.9, 124.4)
- added SW70: DEL, Sony_Hit_Bit:Switch, F.Cu at (277.2, 104.0)
- added SW71: LEFT, Sony_Hit_Bit:Switch, F.Cu at (336.9, 162.5)
- added SW72: UP, Sony_Hit_Bit:Switch, F.Cu at (355.9, 143.4)
- added SW73: DOWN, Sony_Hit_Bit:Switch, F.Cu at (355.9, 181.6)
- added SW74: RIGHT, Sony_Hit_Bit:Switch, F.Cu at (376.0, 162.5)
- added SW8: 7, Sony_Hit_Bit:Switch, F.Cu at (183.9, 124.4)
- added SW9: 8, Sony_Hit_Bit:Switch, F.Cu at (203.0, 124.4)

Commit message: PCB stackup definitions
Other:
- rule pad_to_mask_clearance: 0 -> 0.05
Changed lines of the file:
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@@
 	(generator_version "8.0")
 	(general
-		(thickness 1.6)
+		(thickness 0.244)
 		(legacy_teardrops no)
 	)
@@
 			(layer "F.SilkS"
 				(type "Top Silk Screen")
+				(color "White")
+				(material "Direct Printing")
 			)
 			(layer "F.Paste"
@@
 			(layer "F.Mask"
 				(type "Top Solder Mask")
+				(color "#8080801A")
 				(thickness 0.01)
 			)
 			(layer "F.Cu"
 				(type "copper")
-				(thickness 0.035)
+				(thickness 0.012)
 			)
 			(layer "dielectric 1"
 				(type "core")
-				(thickness 1.51)
-				(material "FR4")
-				(epsilon_r 4.5)
-				(loss_tangent 0.02)
+				(color "Polyimide")
+				(thickness 0.2)
+				(material "Polyimide")
+				(epsilon_r 3.2)
+				(loss_tangent 0.004)
 			)
 			(layer "B.Cu"
 				(type "copper")
-				(thickness 0.035)
+				(thickness 0.012)
 			)
 			(layer "B.Mask"
 				(type "Bottom Solder Mask")
+				(color "#8080801A")
 				(thickness 0.01)
 			)
@@
 			(layer "B.SilkS"
 				(type "Bottom Silk Screen")
+				(color "White")
+				(material "Direct Printing")
 			)
-			(copper_finish "None")
+			(copper_finish "ENIG")
 			(dielectric_constraints no)
 		)
-		(pad_to_mask_clearance 0)
+		(pad_to_mask_clearance 0.05)
+		(solder_mask_min_width 0.25)
 		(allow_soldermask_bridges_in_footprints no)
 		(grid_origin 33.54 213)

Commit message: Track routing
Parts:
- moved J1 0.50 mm to (300.3, 62.0)
- turned SW1 to -135 degrees
- turned SW10 to -135 degrees
- turned SW11 to -135 degrees
- turned SW12 to -135 degrees
- turned SW13 to -135 degrees
- turned SW14 to -135 degrees
- turned SW15 to -135 degrees
- turned SW16 to -135 degrees
- turned SW17 to -135 degrees
- turned SW18 to -135 degrees
- turned SW19 to -135 degrees
- turned SW2 to -135 degrees
- turned SW20 to -135 degrees
- turned SW21 to -135 degrees
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Routing:
- net /5: track 0.00 -> 1027.2 mm, vias 0 -> 4
- net /12: track 0.00 -> 769.5 mm, vias 0 -> 6
- net /9: track 0.00 -> 765.8 mm, vias 0 -> 7
- net /2: track 0.00 -> 704.5 mm, vias 0 -> 6
- net /8: track 0.00 -> 700.9 mm
- net /1: track 0.00 -> 694.7 mm, vias 0 -> 5
- net /7: track 0.00 -> 692.5 mm, vias 0 -> 6
- net /13: track 0.00 -> 690.9 mm, vias 0 -> 5
- net /11: track 0.00 -> 616.8 mm, vias 0 -> 6
- net /10: track 0.00 -> 583.9 mm, vias 0 -> 6
- net /6: track 0.00 -> 520.6 mm, vias 0 -> 2
- net /17: track 0.00 -> 473.1 mm, vias 0 -> 3
- net /15: track 0.00 -> 422.5 mm, vias 0 -> 5
- net /16: track 0.00 -> 411.7 mm, vias 0 -> 5
- net /3: track 0.00 -> 388.7 mm, vias 0 -> 6
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
Commit message: Updating footprints and adding PCB labels
Parts:
- moved J1 0.50 mm to (300.3, 61.5)
Other:
- board text added: "Copyright Alexander Knapik 2025 CERN-OHL-W v2.0 or later"
- board text added: "HB-F1 MSX Keyboard Membrane"

Commit message: PCB fixing position errors and adding labels
Parts:
- added SYM1: Logo_Open_Hardware_Small, Symbol:OSHW-Logo_5.7x6mm_SilkScreen, F.Cu at (310.5, 208.5)
- SW14: value @ -> AT
- SW15: value [ -> LBRACKET
- SW18: value ] -> RBRACKET
- SW21: value / -> SLASH
- SW55: value F1 -> F1/F6
- SW56: value F2 -> F2/F7
- SW57: value F3 -> F3/F8
- SW59: value F4 -> F4/F9
- SW60: value F5 -> F5/F10
- moved SW74 1.00 mm to (375.0, 162.5)
- turned SW55 to 90 degrees
Routing:
- net Net-(J1-Pin_21): track 155.2 -> 236.5 mm, vias 2 -> 0
- net Net-(J1-Pin_22): track 167.4 -> 247.3 mm, vias 2 -> 0
- net /5: track 1027.2 -> 1030.1 mm
- net /8: track 700.9 -> 698.8 mm
- net /2: track 704.5 -> 703.5 mm
- net Net-(D1-K): track 70.0 -> 69.4 mm
- net Net-(D1-A): track 65.8 -> 65.2 mm
Other:
- rule pad_to_mask_clearance: 0.05 -> 0
- board text added: "+"
- board text added: "CERN-OHL-W v2 or later"
- board text added: "Copyright Alexander Knapik 2025"
- board text added: "POWER"
- board text added: "−"
- board text removed: "Copyright Alexander Knapik 2025 CERN-OHL-W v2.0 or later"

Commit message: PCB adding fiducials
Parts:
- added FID1: Fiducial, Fiducial:Fiducial_1mm_Mask2mm, F.Cu at (35.5, 211.0)
- added FID2: Fiducial, Fiducial:Fiducial_1mm_Mask2mm, F.Cu at (381.5, 101.5)
